Commit message: completed simple move_base function

File: racecar_simulator/urdf/move_macro.xacro (robot description, xacro)
@@ -10,5 +10,4 @@
       <child  link="${prefix}_link"/>
       <axis xyz="0 0 1" />
-      <anchor xyz="0 0 0"/>
       <limit velocity="200" effort="200" />
       <dynamics damping="0.1"/>
@@ -27,5 +26,5 @@
       <inertial>
         <origin xyz="0 0 0" rpy="0 0 0"/>
-        <mass value="0.1"/>
+        <mass value="1.5"/>
         <inertia ixx="0.0001" ixy="0.0" ixz="0.0" iyy="0.0001" iyz="0.0" izz="0.0001"/>
       </inertial>
@@ -60,5 +59,5 @@
     <link name="body_link">
       <inertial>
-        <mass value="1.0"/>
+        <mass value="15.0"/>
         <origin xyz=" 0 0 0.1175"/>
         <inertia ixx="0.001" ixy="0.0" ixz="0.0" iyy="0.001" iyz="0.0" izz="0.001"/>

File: racecar_simulator/urdf/racecar.xacro (robot description, xacro)
@@ -223,9 +223,4 @@
   <!-- Laser -->
   <link name="laser">
-   <inertial>
-      <mass value="1e-5" />
-      <origin xyz="0 0 0" rpy="0 0 0"/>
-      <inertia ixx="1e-6" ixy="0" ixz="0" iyy="1e-6" iyz="0" izz="1e-6" />
-    </inertial>
     <collision>
       <origin rpy="0 0 0" xyz="0 0 0"/>
@@ -266,9 +261,9 @@
           <resolution>0.01</resolution>
         </range>
-        <!--noise>
+        <noise>
           <type>gaussian</type>
           <mean>0.0</mean>
           <stddev>0.001</stddev>
-        </noise-->
+        </noise>
       </ray>
       <plugin name="gazebo_laser_controller" filename="libgazebo_ros_laser.so">
@@ -281,9 +276,4 @@
   <!-- IMU -->
   <link name="IMU_link">
-   <inertial>
-      <mass value="1e-5" />
-      <origin xyz="0 0 0" rpy="0 0 0"/>
-      <inertia ixx="1e-6" ixy="0" ixz="0" iyy="1e-6" iyz="0" izz="1e-6" />
-    </inertial>
     <collision>
       <origin rpy="0 0 0" xyz="0 0 0"/>

File: racecar_simulator/urdf/racecar_robot.xacro (robot description, xacro)
@@ -2,4 +2,7 @@
 <robot name="racecar" xmlns:xacro="http://ros.org/wiki/xacro">
   <xacro:arg name="robot_name" default="racecar"/>
+  <xacro:arg name="enable_odom_tf" default="true"/>
+  <xacro:arg name="odom_frame" default="odom"/>
+  <xacro:arg name="odom_topic" default="odom"/>
   <xacro:include filename="$(find racecar_simulator)/urdf/move_macro.xacro"/>
   <xacro:include filename="$(find racecar_simulator)/urdf/laser_macro.xacro"/>
@@ -14,8 +17,23 @@
   <xacro:imu_macro prefix="imu" parent="base_link" xyz="0.16575 0 0.168" robot_name="$(arg robot_name)"/>
   <gazebo>
-    <plugin name="gazebo_ros_control" filename="libgazebo_ros_control.so">
+    <plugin filename="libgazebo_ros_skid_steer_drive.so" name="skid_steer_drive_controller">
+      <updateRate>100.0</updateRate>
       <robotNamespace>$(arg robot_name)</robotNamespace>
-      <robotSimType>gazebo_ros_control/DefaultRobotHWSim</robotSimType>
-      <legacyModeNS>true</legacyModeNS>
+      <leftFrontJoint>front_left_wheel_joint</leftFrontJoint>
+      <rightFrontJoint>front_right_wheel_joint</rightFrontJoint>
+      <leftRearJoint>rear_left_wheel_joint</leftRearJoint>
+      <rightRearJoint>rear_right_wheel_joint</rightRearJoint>
+      <covariance_x>0.000100</covariance_x>
+      <covariance_y>0.000100</covariance_y>
+      <covariance_yaw>0.010000</covariance_yaw>
+      <wheelSeparation>0.28</wheelSeparation>
+      <wheelDiameter>0.135</wheelDiameter>
+      <robotBaseFrame>$(arg robot_name)/base_link</robotBaseFrame>
+      <MaxForce>10.0</MaxForce>
+      <torque>400</torque>
+      <commandTopic>cmd_vel</commandTopic>
+      <odometryTopic>$(arg odom_topic)</odometryTopic>
+      <odometryFrame>$(arg robot_name)/$(arg odom_frame)</odometryFrame>
+      <broadcastTF>$(arg enable_odom_tf)</broadcastTF>
     </plugin>
   </gazebo>

Commit message: edited *.launch files

File: racecar_simulator/urdf/move_macro.xacro (robot description, xacro)
@@ -26,5 +26,5 @@
       <inertial>
         <origin xyz="0 0 0" rpy="0 0 0"/>
-        <mass value="1.5"/>
+        <mass value="0.1"/>
         <inertia ixx="0.0001" ixy="0.0" ixz="0.0" iyy="0.0001" iyz="0.0" izz="0.0001"/>
       </inertial>
@@ -59,5 +59,5 @@
     <link name="body_link">
       <inertial>
-        <mass value="15.0"/>
+        <mass value="1.0"/>
         <origin xyz=" 0 0 0.1175"/>
         <inertia ixx="0.001" ixy="0.0" ixz="0.0" iyy="0.001" iyz="0.0" izz="0.001"/>

File: racecar_simulator/urdf/racecar.xacro (robot description, xacro)
@@ -1,13 +1,18 @@
 <?xml version="1.0"?>
 <robot name="racecar" xmlns:xacro="http://www.ros.org/wiki/xacro">
+  <xacro:arg name="robot_name" default="racecar"/>
+  <xacro:arg name="enable_odom_tf" default="true"/>
+  <xacro:arg name="odom_frame" default="odom"/>
+  <xacro:arg name="odom_topic" default="odom"/>
   <material name="white">
     <color rgba="1.0 1.0 1.0 1.0"/>
   </material>
+  <link name="base_link"/>
   <!-- Chassis -->
-  <link name="base_footprint">
-    <inertial>
-      <mass value="1.0"/>
+  <link name="body_link">
+    <inertial>
+      <mass value="15.0"/>
       <origin xyz=" 0 0 0.1175"/>
-      <inertia ixx="0.001" ixy="0.0" ixz="0.0" iyy="0.001" iyz="0.0" izz="0.001"/>
+      <inertia ixx="0.13" ixy="0.0" ixz="0.0" iyy="0.33" iyz="0.0" izz="0.39"/>
     </inertial>
     <visual>
@@ -25,5 +30,10 @@
     </collision>
   </link>
-  <gazebo reference="base_footprint">
+  <joint name="body_joint" type="fixed">
+    <parent link="base_link"/>
+    <child  link="body_link"/>
+    <origin xyz="0 0 0" rpy="0 0 0"/>
+  </joint>
+  <gazebo reference="body_link">
     <material value="Gazebo/White"/>
   </gazebo>
@@ -32,6 +42,6 @@
     <inertial>
       <origin xyz="0 0 0" rpy="0 0 0"/>
-      <mass value="0.1"/>
-      <inertia ixx="0.0001" ixy="0.0" ixz="0.0" iyy="0.0001" iyz="0.0" izz="0.0001"/>
+      <mass value="1.5"/>
+      <inertia ixx="0.005" ixy="0.0" ixz="0.0" iyy="0.005" iyz="0.0" izz="0.009"/>
     </inertial>
     <visual>
@@ -55,5 +65,5 @@
     <joint_properties damping="0.1"/>
     <origin rpy="${radians(-90)} 0 0" xyz="0.1575 0.14 0.0675"/>
-    <parent link="base_footprint"/>
+    <parent link="base_link"/>
     <child link="front_left_wheel_link"/>
   </joint>
@@ -61,5 +71,5 @@
     <type>transmission_interface/SimpleTransmission</type>
     <joint name="front_left_wheel_joint">
-        <hardwareInterface>hardware_interface/VelocityJointInterface</hardwareInterface>
+      <hardwareInterface>hardware_interface/VelocityJointInterface</hardwareInterface>
     </joint>
     <actuator name="$front_left_wheel_motor">
@@ -80,6 +90,6 @@
     <inertial>
       <origin xyz="0 0 0" rpy="0 0 0"/>
-      <mass value="0.1"/>
-      <inertia ixx="0.0001" ixy="0.0" ixz="0.0" iyy="0.0001" iyz="0.0" izz="0.0001"/>
+      <mass value="1.5"/>
+      <inertia ixx="0.005" ixy="0.0" ixz="0.0" iyy="0.005" iyz="0.0" izz="0.009"/>
     </inertial>
     <visual>
@@ -103,5 +113,5 @@
     <joint_properties damping="0.1"/>
     <origin rpy="${radians(-90)} 0 0" xyz="-0.1575 0.14 0.0675"/>
-    <parent link="base_footprint"/>
+    <parent link="base_link"/>
     <child link="rear_left_wheel_link"/>
   </joint>
@@ -109,5 +119,5 @@
     <type>transmission_interface/SimpleTransmission</type>
     <joint name="rear_left_wheel_joint">
-        <hardwareInterface>hardware_interface/VelocityJointInterface</hardwareInterface>
+      <hardwareInterface>hardware_interface/VelocityJointInterface</hardwareInterface>
     </joint>
     <actuator name="rear_left_wheel_motor">
@@ -128,6 +138,6 @@
     <inertial>
       <origin xyz="0 0 0" rpy="0 0 0"/>
-      <mass value="0.1"/>
-      <inertia ixx="0.0001" ixy="0.0" ixz="0.0" iyy="0.0001" iyz="0.0" izz="0.0001"/>
+      <mass value="1.5"/>
+      <inertia ixx="0.005" ixy="0.0" ixz="0.0" iyy="0.005" iyz="0.0" izz="0.009"/>
     </inertial>
     <visual>
@@ -151,5 +161,5 @@
     <joint_properties damping="0.1"/>
     <origin rpy="${radians(-90)} 0 0" xyz="0.1575 -0.14 0.0675"/>
-    <parent link="base_footprint"/>
+    <parent link="base_link"/>
     <child link="front_right_wheel_link"/>
   </joint>
@@ -157,5 +167,5 @@
     <type>transmission_interface/SimpleTransmission</type>
     <joint name="front_right_wheel_joint">
-        <hardwareInterface>hardware_interface/VelocityJointInterface</hardwareInterface>
+      <hardwareInterface>hardware_interface/VelocityJointInterface</hardwareInterface>
     </joint>
     <actuator name="front_right_wheel_motor">
@@ -176,6 +186,6 @@
     <inertial>
       <origin xyz="0 0 0" rpy="0 0 0"/>
-      <mass value="0.1"/>
-      <inertia ixx="0.0001" ixy="0.0" ixz="0.0" iyy="0.0001" iyz="0.0" izz="0.0001"/>
+      <mass value="1.5"/>
+      <inertia ixx="0.005" ixy="0.0" ixz="0.0" iyy="0.005" iyz="0.0" izz="0.009"/>
     </inertial>
     <visual>
@@ -199,5 +209,5 @@
     <joint_properties damping="0.1"/>
     <origin rpy="${radians(-90)} 0 0" xyz="-0.1575 -0.14 0.0675"/>
-    <parent link="base_footprint"/>
+    <parent link="base_link"/>
     <child link="rear_right_wheel_link"/>
   </joint>
@@ -205,5 +215,5 @@
     <type>transmission_interface/SimpleTransmission</type>
     <joint name="rear_right_wheel_joint">
-        <hardwareInterface>hardware_interface/VelocityJointInterface</hardwareInterface>
+      <hardwareInterface>hardware_interface/VelocityJointInterface</hardwareInterface>
     </joint>
     <actuator name="rear_right_wheel_motor">
@@ -222,5 +232,5 @@
   </gazebo>
   <!-- Laser -->
-  <link name="laser">
+  <link name="laser_link">
     <collision>
       <origin rpy="0 0 0" xyz="0 0 0"/>
@@ -239,8 +249,8 @@
   <joint name="laser_joint" type="fixed">
     <origin rpy="0 0 0" xyz="0.07 0 0.2575"/>
-    <parent link="base_footprint"/>
-    <child link="laser"/>
-  </joint>
-  <gazebo reference="laser">
+    <parent link="base_link"/>
+    <child link="laser_link"/>
+  </joint>
+  <gazebo reference="laser_link">
     <sensor type="ray" name="art_laser">
       <pose>0 0 0.0175 0 0 0</pose>
@@ -268,5 +278,5 @@
       </ray>
       <plugin name="gazebo_laser_controller" filename="libgazebo_ros_laser.so">
-        <topicName>/scan</topicName>
+        <topicName>laser/scan</topicName>
         <frameName>laser</frameName>
       </plugin>
@@ -275,5 +285,5 @@
   </gazebo>
   <!-- IMU -->
-  <link name="IMU_link">
+  <link name="imu_link">
     <collision>
       <origin rpy="0 0 0" xyz="0 0 0"/>
@@ -292,8 +302,8 @@
   <joint name="imu_joint" type="fixed">
     <origin rpy="0 0 0" xyz="0.16575 0 0.168"/>
-    <parent link="base_footprint"/>
-    <child link="IMU_link"/>
-  </joint>
-  <gazebo reference="IMU_link">
+    <parent link="base_link"/>
+    <child link="imu_link"/>
+  </joint>
+  <gazebo reference="imu_link">
     <pose>0 0 0.01 0 0 0</pose>
     <gravity>true</gravity>
@@ -302,13 +312,13 @@
       <update_rate>100</update_rate>
       <visualize>true</visualize>
-      <topic>__default_topic__</topic>
+      <topic>data</topic>
       <plugin filename="libgazebo_ros_imu_sensor.so" name="imu_plugin">
-        <topicName>/imu_data</topicName>
-        <bodyName>IMU_link</bodyName>
+        <topicName>/imu/data</topicName>
+        <bodyName>imu_link</bodyName>
         <updateRateHZ>100.0</updateRateHZ>
         <gaussianNoise>0.0</gaussianNoise>
         <xyzOffset>0 0 0</xyzOffset>
         <rpyOffset>0 0 0</rpyOffset>
-        <frameName>IMU_link</frameName>
+        <frameName>$(arg robot_name)/imu_link</frameName>
       </plugin>
     </sensor>
@@ -317,5 +327,5 @@
   <!-- Plugin -->
   <gazebo>
-    <!--plugin filename="libgazebo_ros_skid_steer_drive.so" name="skid_steer_drive_controller">
+    <plugin filename="libgazebo_ros_skid_steer_drive.so" name="skid_steer_drive_controller">
       <updateRate>100.0</updateRate>
       <robotNamespace>$(arg robot_name)</robotNamespace>
@@ -324,14 +334,17 @@
       <leftRearJoint>rear_left_wheel_joint</leftRearJoint>
       <rightRearJoint>rear_right_wheel_joint</rightRearJoint>
-      <wheelSeparation>0.315</wheelSeparation>
+      <covariance_x>0.000100</covariance_x>
+      <covariance_y>0.000100</covariance_y>
+      <covariance_yaw>0.010000</covariance_yaw>
+      <wheelSeparation>0.28</wheelSeparation>
       <wheelDiameter>0.135</wheelDiameter>
-      <robotBaseFrame>racecar/base_link</robotBaseFrame>
+      <robotBaseFrame>$(arg robot_name)/base_link</robotBaseFrame>
       <MaxForce>10.0</MaxForce>
       <torque>400</torque>
       <commandTopic>cmd_vel</commandTopic>
-      <odometryTopic>odom</odometryTopic>
-      <odometryFrame>odom</odometryFrame>
-      <broadcastTF>1</broadcastTF>
-    </plugin-->
+      <odometryTopic>$(arg odom_topic)</odometryTopic>
+      <odometryFrame>$(arg robot_name)/$(arg odom_frame)</odometryFrame>
+      <broadcastTF>$(arg enable_odom_tf)</broadcastTF>
+    </plugin>
     <!--plugin name="object_controller" filename="libgazebo_ros_planar_move.so">
       <commandTopic>cmd_vel</commandTopic>
@@ -339,11 +352,11 @@
       <odometryFrame>odom</odometryFrame>
       <odometryRate>20.0</odometryRate>
-      <robotBaseFrame>base_footprint</robotBaseFrame>
+      <robotBaseFrame>base_link</robotBaseFrame>
     </plugin-->
-    <plugin name="gazebo_ros_control" filename="libgazebo_ros_control.so">
+    <!--plugin name="gazebo_ros_control" filename="libgazebo_ros_control.so">
       <robotNamespace>$(arg robot_name)</robotNamespace>
       <robotSimType>gazebo_ros_control/DefaultRobotHWSim</robotSimType>
       <legacyModeNS>true</legacyModeNS>
-    </plugin>
+    </plugin-->
   </gazebo>
 </robot>

File: racecar_simulator/urdf/racecar_robot.xacro (robot description, xacro)
@@ -37,4 +37,11 @@
       <broadcastTF>$(arg enable_odom_tf)</broadcastTF>
     </plugin>
+    <!--plugin name="object_controller" filename="libgazebo_ros_planar_move.so">
+      <commandTopic>cmd_vel</commandTopic>
+      <odometryTopic>odom</odometryTopic>
+      <odometryFrame>$(arg robot_name)/odom</odometryFrame>
+      <odometryRate>100.0</odometryRate>
+      <robotBaseFrame>$(arg robot_name)/base_link</robotBaseFrame>
+    </plugin-->
   </gazebo>
 </robot>
