Commit message: fix param setup problems in dwa_local_planner

File: racecar_simulator/urdf/move_macro.xacro (robot description, xacro)
@@ -24,4 +24,11 @@
     </transmission>
     <link name="${prefix}_link">
+      <!-- libgazebo_ros_planar_move.so -->
+      <!--inertial>
+      <origin xyz="0 0 0" rpy="0 0 0"/>
+      <mass value="1.5"/>
+      <inertia ixx="0.005" ixy="0.0" ixz="0.0" iyy="0.005" iyz="0.0" izz="0.009"/>
+      </inertial-->
+      <!--libgazebo_ros_skid_steer_drive.so -->
       <inertial>
         <origin xyz="0 0 0" rpy="0 0 0"/>
@@ -49,4 +56,5 @@
       <kp value="50000" />
       <kd value="10" />
+      <minDepth>0.00</minDepth>
     </gazebo>
   </xacro:macro>
@@ -58,4 +66,11 @@
     </joint>
     <link name="body_link">
+      <!-- libgazebo_ros_planar_move.so -->
+      <!--inertial>
+      <mass value="15.0"/>
+      <origin xyz=" 0 0 0.1175"/>
+      <inertia ixx="0.13" ixy="0.0" ixz="0.0" iyy="0.33" iyz="0.0" izz="0.39"/>
+      </inertial-->
+      <!--libgazebo_ros_skid_steer_drive.so -->
       <inertial>
         <mass value="1.0"/>

File: racecar_simulator/urdf/racecar.xacro (robot description, xacro)
@@ -1,18 +1,13 @@
 <?xml version="1.0"?>
-<robot name="racecar" xmlns:xacro="http://www.ros.org/wiki/xacro">
-  <xacro:arg name="robot_name" default="racecar"/>
-  <xacro:arg name="enable_odom_tf" default="true"/>
-  <xacro:arg name="odom_frame" default="odom"/>
-  <xacro:arg name="odom_topic" default="odom"/>
+<robot name="rrbot" xmlns:xacro="http://www.ros.org/wiki/xacro">
   <material name="white">
     <color rgba="1.0 1.0 1.0 1.0"/>
   </material>
-  <link name="base_link"/>
   <!-- Chassis -->
-  <link name="body_link">
-    <inertial>
-      <mass value="15.0"/>
+  <link name="base_link">
+    <inertial>
+      <mass value="21.5"/>
       <origin xyz=" 0 0 0.1175"/>
-      <inertia ixx="0.13" ixy="0.0" ixz="0.0" iyy="0.33" iyz="0.0" izz="0.39"/>
+      <inertia ixx="0.3338" ixy="0.0" ixz="0.0" iyy="0.4783" iyz="0.0" izz="0.3338"/>
     </inertial>
     <visual>
@@ -30,28 +25,23 @@
     </collision>
   </link>
-  <joint name="body_joint" type="fixed">
-    <parent link="base_link"/>
-    <child  link="body_link"/>
-    <origin xyz="0 0 0" rpy="0 0 0"/>
-  </joint>
-  <gazebo reference="body_link">
+  <gazebo reference="base_link">
     <material value="Gazebo/White"/>
   </gazebo>
   <!-- wheel -->
-  <link name="front_left_wheel_link">
-    <inertial>
-      <origin xyz="0 0 0" rpy="0 0 0"/>
-      <mass value="1.5"/>
-      <inertia ixx="0.005" ixy="0.0" ixz="0.0" iyy="0.005" iyz="0.0" izz="0.009"/>
-    </inertial>
-    <visual>
-      <origin rpy="0 0 0" xyz="0 0 0"/>
-      <geometry>
-        <cylinder radius="0.0675" length="0.064"/>
-      </geometry>
-      <material name="white"/>
-    </visual>
-    <collision>
-      <origin rpy="0 0 0" xyz="0 0 0"/>
+  <link name="front_left_wheel">
+    <inertial>
+      <mass value="1.2"/>
+      <origin xyz="0 0 0"/>
+      <inertia ixx="0.01241176559" ixy="0" ixz="0" iyy="0.01521816042" iyz="0" izz="0.01176397794"/>
+    </inertial>
+    <visual>
+      <origin rpy="-1.5707 0 0" xyz="0 0 0"/>
+      <geometry>
+        <cylinder radius="0.0675" length="0.064"/>
+      </geometry>
+      <material name="white"/>
+    </visual>
+    <collision>
+      <origin rpy="-1.5707 0 0" xyz="0 0 0"/>
       <geometry>
         <cylinder radius="0.0675" length="0.064"/>
@@ -60,23 +50,13 @@
   </link>
   <joint name="front_left_wheel_joint" type="continuous">
-    <axis xyz="0 0 1"/>
+    <axis xyz="0 1 0"/>
     <anchor xyz="0 0 0"/>
     <limit effort="200" velocity="200"/>
-    <joint_properties damping="0.1"/>
-    <origin rpy="${radians(-90)} 0 0" xyz="0.1575 0.14 0.0675"/>
-    <parent link="base_link"/>
-    <child link="front_left_wheel_link"/>
-  </joint>
-  <transmission name="front_left_wheel_trans">
-    <type>transmission_interface/SimpleTransmission</type>
-    <joint name="front_left_wheel_joint">
-      <hardwareInterface>hardware_interface/VelocityJointInterface</hardwareInterface>
-    </joint>
-    <actuator name="$front_left_wheel_motor">
-      <hardwareInterface>hardware_interface/VelocityJointInterface</hardwareInterface>
-      <mechanismReduction>1</mechanismReduction>
-    </actuator>
-  </transmission>
-  <gazebo reference="front_left_wheel_link">
+    <joint_properties damping="0.7"/>
+    <origin rpy="0 0 0" xyz="0.1575 0.14 0.0675"/>
+    <parent link="base_link"/>
+    <child link="front_left_wheel"/>
+  </joint>
+  <gazebo reference="front_left_wheel">
     <kp>1000000.0</kp>
     <kd>100.0</kd>
@@ -87,19 +67,19 @@
     <material value="Gazebo/White"/>
   </gazebo>
-  <link name="rear_left_wheel_link">
-    <inertial>
-      <origin xyz="0 0 0" rpy="0 0 0"/>
-      <mass value="1.5"/>
-      <inertia ixx="0.005" ixy="0.0" ixz="0.0" iyy="0.005" iyz="0.0" izz="0.009"/>
-    </inertial>
-    <visual>
-      <origin rpy="0 0 0" xyz="0 0 0"/>
-      <geometry>
-        <cylinder radius="0.0675" length="0.064"/>
-      </geometry>
-      <material name="white"/>
-    </visual>
-    <collision>
-      <origin rpy="0 0 0" xyz="0 0 0"/>
+  <link name="rear_left_wheel">
+    <inertial>
+      <mass value="1.2"/>
+      <origin xyz="0 0 0"/>
+      <inertia ixx="0.01241176559" ixy="0" ixz="0" iyy="0.01521816042" iyz="0" izz="0.01176397794"/>
+    </inertial>
+    <visual>
+      <origin rpy="-1.5707 0 0" xyz="0 0 0"/>
+      <geometry>
+        <cylinder radius="0.0675" length="0.064"/>
+      </geometry>
+      <material name="white"/>
+    </visual>
+    <collision>
+      <origin rpy="-1.5707 0 0" xyz="0 0 0"/>
       <geometry>
         <cylinder radius="0.0675" length="0.064"/>
@@ -108,23 +88,13 @@
   </link>
   <joint name="rear_left_wheel_joint" type="continuous">
-    <axis xyz="0 0 1"/>
+    <axis xyz="0 1 0"/>
     <anchor xyz="0 0 0"/>
     <limit effort="200" velocity="200"/>
-    <joint_properties damping="0.1"/>
-    <origin rpy="${radians(-90)} 0 0" xyz="-0.1575 0.14 0.0675"/>
-    <parent link="base_link"/>
-    <child link="rear_left_wheel_link"/>
-  </joint>
-  <transmission name="rear_left_wheel_trans">
-    <type>transmission_interface/SimpleTransmission</type>
-    <joint name="rear_left_wheel_joint">
-      <hardwareInterface>hardware_interface/VelocityJointInterface</hardwareInterface>
-    </joint>
-    <actuator name="rear_left_wheel_motor">
-      <hardwareInterface>hardware_interface/VelocityJointInterface</hardwareInterface>
-      <mechanismReduction>1</mechanismReduction>
-    </actuator>
-  </transmission>
-  <gazebo reference="rear_left_wheel_link">
+    <joint_properties damping="0.7"/>
+    <origin rpy="0 0 0" xyz="-0.1575 0.14 0.0675"/>
+    <parent link="base_link"/>
+    <child link="rear_left_wheel"/>
+  </joint>
+  <gazebo reference="rear_left_wheel">
     <kp>1000000.0</kp>
     <kd>100.0</kd>
@@ -135,19 +105,19 @@
     <material value="Gazebo/White"/>
   </gazebo>
-  <link name="front_right_wheel_link">
-    <inertial>
-      <origin xyz="0 0 0" rpy="0 0 0"/>
-      <mass value="1.5"/>
-      <inertia ixx="0.005" ixy="0.0" ixz="0.0" iyy="0.005" iyz="0.0" izz="0.009"/>
-    </inertial>
-    <visual>
-      <origin rpy="0 0 0" xyz="0 0 0"/>
-      <geometry>
-        <cylinder radius="0.0675" length="0.064"/>
-      </geometry>
-      <material name="white"/>
-    </visual>
-    <collision>
-      <origin rpy="0 0 0" xyz="0 0 0"/>
+  <link name="front_right_wheel">
+    <inertial>
+      <mass value="1.2"/>
+      <origin xyz="0 0 0"/>
+      <inertia ixx="0.01241176559" ixy="0" ixz="0" iyy="0.01521816042" iyz="0" izz="0.01176397794"/>
+    </inertial>
+    <visual>
+      <origin rpy="-1.5707 0 0" xyz="0 0 0"/>
+      <geometry>
+        <cylinder radius="0.0675" length="0.064"/>
+      </geometry>
+      <material name="white"/>
+    </visual>
+    <collision>
+      <origin rpy="-1.5707 0 0" xyz="0 0 0"/>
       <geometry>
         <cylinder radius="0.0675" length="0.064"/>
@@ -156,23 +126,13 @@
   </link>
   <joint name="front_right_wheel_joint" type="continuous">
-    <axis xyz="0 0 1"/>
+    <axis xyz="0 1 0"/>
     <anchor xyz="0 0 0"/>
     <limit effort="200" velocity="200"/>
-    <joint_properties damping="0.1"/>
-    <origin rpy="${radians(-90)} 0 0" xyz="0.1575 -0.14 0.0675"/>
-    <parent link="base_link"/>
-    <child link="front_right_wheel_link"/>
-  </joint>
-  <transmission name="front_right_wheel_trans">
-    <type>transmission_interface/SimpleTransmission</type>
-    <joint name="front_right_wheel_joint">
-      <hardwareInterface>hardware_interface/VelocityJointInterface</hardwareInterface>
-    </joint>
-    <actuator name="front_right_wheel_motor">
-      <hardwareInterface>hardware_interface/VelocityJointInterface</hardwareInterface>
-      <mechanismReduction>1</mechanismReduction>
-    </actuator>
-  </transmission>
-  <gazebo reference="front_right_wheel_link">
+    <joint_properties damping="0.7"/>
+    <origin rpy="0 0 0" xyz="0.1575 -0.14 0.0675"/>
+    <parent link="base_link"/>
+    <child link="front_right_wheel"/>
+  </joint>
+  <gazebo reference="front_right_wheel">
     <kp>1000000.0</kp>
     <kd>100.0</kd>
@@ -183,19 +143,19 @@
     <material value="Gazebo/White"/>
   </gazebo>
-  <link name="rear_right_wheel_link">
-    <inertial>
-      <origin xyz="0 0 0" rpy="0 0 0"/>
-      <mass value="1.5"/>
-      <inertia ixx="0.005" ixy="0.0" ixz="0.0" iyy="0.005" iyz="0.0" izz="0.009"/>
-    </inertial>
-    <visual>
-      <origin rpy="0 0 0" xyz="0 0 0"/>
-      <geometry>
-        <cylinder radius="0.0675" length="0.064"/>
-      </geometry>
-      <material name="white"/>
-    </visual>
-    <collision>
-      <origin rpy="0 0 0" xyz="0 0 0"/>
+  <link name="rear_right_wheel">
+    <inertial>
+      <mass value="1.2"/>
+      <origin xyz="0 0 0"/>
+      <inertia ixx="0.01241176559" ixy="0" ixz="0" iyy="0.01521816042" iyz="0" izz="0.01176397794"/>
+    </inertial>
+    <visual>
+      <origin rpy="-1.5707 0 0" xyz="0 0 0"/>
+      <geometry>
+        <cylinder radius="0.0675" length="0.064"/>
+      </geometry>
+      <material name="white"/>
+    </visual>
+    <collision>
+      <origin rpy="-1.5707 0 0" xyz="0 0 0"/>
       <geometry>
         <cylinder radius="0.0675" length="0.064"/>
@@ -204,23 +164,13 @@
   </link>
   <joint name="rear_right_wheel_joint" type="continuous">
-    <axis xyz="0 0 1"/>
+    <axis xyz="0 1 0"/>
     <anchor xyz="0 0 0"/>
     <limit effort="200" velocity="200"/>
-    <joint_properties damping="0.1"/>
-    <origin rpy="${radians(-90)} 0 0" xyz="-0.1575 -0.14 0.0675"/>
-    <parent link="base_link"/>
-    <child link="rear_right_wheel_link"/>
-  </joint>
-  <transmission name="rear_right_wheel_trans">
-    <type>transmission_interface/SimpleTransmission</type>
-    <joint name="rear_right_wheel_joint">
-      <hardwareInterface>hardware_interface/VelocityJointInterface</hardwareInterface>
-    </joint>
-    <actuator name="rear_right_wheel_motor">
-      <hardwareInterface>hardware_interface/VelocityJointInterface</hardwareInterface>
-      <mechanismReduction>1</mechanismReduction>
-    </actuator>
-  </transmission>
-  <gazebo reference="rear_right_wheel_link">
+    <joint_properties damping="0.7"/>
+    <origin rpy="0 0 0" xyz="-0.1575 -0.14 0.0675"/>
+    <parent link="base_link"/>
+    <child link="rear_right_wheel"/>
+  </joint>
+  <gazebo reference="rear_right_wheel">
     <kp>1000000.0</kp>
     <kd>100.0</kd>
@@ -233,4 +183,9 @@
   <!-- Laser -->
   <link name="laser_link">
+   <inertial>
+      <mass value="1e-5" />
+      <origin xyz="0 0 0" rpy="0 0 0"/>
+      <inertia ixx="1e-6" ixy="0" ixz="0" iyy="1e-6" iyz="0" izz="1e-6" />
+    </inertial>
     <collision>
       <origin rpy="0 0 0" xyz="0 0 0"/>
@@ -256,5 +211,5 @@
       <pose>0 0 0.0175 0 0 0</pose>
       <visualize>false</visualize>
-      <update_rate>10</update_rate>
+      <update_rate>11</update_rate>
       <ray>
         <scan>
@@ -262,6 +217,6 @@
             <samples>360</samples>
             <resolution>1</resolution>
-            <min_angle>${radians(-180)}</min_angle>
-            <max_angle>${radians(180)}</max_angle>
+            <min_angle>0</min_angle>
+            <max_angle>6.283185</max_angle>
           </horizontal>
         </scan>
@@ -278,6 +233,6 @@
       </ray>
       <plugin name="gazebo_laser_controller" filename="libgazebo_ros_laser.so">
-        <topicName>laser/scan</topicName>
-        <frameName>laser</frameName>
+        <topicName>/laser/scan</topicName>
+        <frameName>laser_link</frameName>
       </plugin>
     </sensor>
@@ -286,4 +241,9 @@
   <!-- IMU -->
   <link name="imu_link">
+   <inertial>
+      <mass value="1e-5" />
+      <origin xyz="0 0 0" rpy="0 0 0"/>
+      <inertia ixx="1e-6" ixy="0" ixz="0" iyy="1e-6" iyz="0" izz="1e-6" />
+    </inertial>
     <collision>
       <origin rpy="0 0 0" xyz="0 0 0"/>
@@ -312,5 +272,5 @@
       <update_rate>100</update_rate>
       <visualize>true</visualize>
-      <topic>data</topic>
+      <topic>__default_topic__</topic>
       <plugin filename="libgazebo_ros_imu_sensor.so" name="imu_plugin">
         <topicName>/imu/data</topicName>
@@ -320,5 +280,5 @@
         <xyzOffset>0 0 0</xyzOffset>
         <rpyOffset>0 0 0</rpyOffset>
-        <frameName>$(arg robot_name)/imu_link</frameName>
+        <frameName>imu_link</frameName>
       </plugin>
     </sensor>
@@ -327,36 +287,28 @@
   <!-- Plugin -->
   <gazebo>
-    <plugin filename="libgazebo_ros_skid_steer_drive.so" name="skid_steer_drive_controller">
+    <!--plugin filename="libgazebo_ros_skid_steer_drive.so" name="skid_steer_drive_controller">
       <updateRate>100.0</updateRate>
-      <robotNamespace>$(arg robot_name)</robotNamespace>
+      <robotNamespace></robotNamespace>
       <leftFrontJoint>front_left_wheel_joint</leftFrontJoint>
       <rightFrontJoint>front_right_wheel_joint</rightFrontJoint>
       <leftRearJoint>rear_left_wheel_joint</leftRearJoint>
       <rightRearJoint>rear_right_wheel_joint</rightRearJoint>
-      <covariance_x>0.000100</covariance_x>
-      <covariance_y>0.000100</covariance_y>
-      <covariance_yaw>0.010000</covariance_yaw>
-      <wheelSeparation>0.28</wheelSeparation>
+      <wheelSeparation>0.34</wheelSeparation>
       <wheelDiameter>0.135</wheelDiameter>
-      <robotBaseFrame>$(arg robot_name)/base_link</robotBaseFrame>
+      <robotBaseFrame>base_link</robotBaseFrame>
       <MaxForce>10.0</MaxForce>
       <torque>400</torque>
       <commandTopic>cmd_vel</commandTopic>
-      <odometryTopic>$(arg odom_topic)</odometryTopic>
-      <odometryFrame>$(arg robot_name)/$(arg odom_frame)</odometryFrame>
-      <broadcastTF>$(arg enable_odom_tf)</broadcastTF>
-    </plugin>
-    <!--plugin name="object_controller" filename="libgazebo_ros_planar_move.so">
+      <odometryTopic>odom</odometryTopic>
+      <odometryFrame>odom</odometryFrame>
+      <broadcastTF>1</broadcastTF>
+    </plugin-->
+    <plugin name="object_controller" filename="libgazebo_ros_planar_move.so">
       <commandTopic>cmd_vel</commandTopic>
       <odometryTopic>odom</odometryTopic>
       <odometryFrame>odom</odometryFrame>
-      <odometryRate>20.0</odometryRate>
+      <odometryRate>100.0</odometryRate>
       <robotBaseFrame>base_link</robotBaseFrame>
-    </plugin-->
-    <!--plugin name="gazebo_ros_control" filename="libgazebo_ros_control.so">
-      <robotNamespace>$(arg robot_name)</robotNamespace>
-      <robotSimType>gazebo_ros_control/DefaultRobotHWSim</robotSimType>
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
Commit message: created a libgazebo_ros_planar_move_drive to control model

File: racecar_simulator/urdf/move_macro.xacro (robot description, xacro)
@@ -11,5 +11,4 @@
       <axis xyz="0 0 1" />
       <limit velocity="200" effort="200" />
-      <dynamics damping="0.1"/>
     </joint>
     <transmission name="${prefix}_trans">
@@ -24,15 +23,8 @@
     </transmission>
     <link name="${prefix}_link">
-      <!-- libgazebo_ros_planar_move.so -->
-      <!--inertial>
+      <inertial>
       <origin xyz="0 0 0" rpy="0 0 0"/>
       <mass value="1.5"/>
       <inertia ixx="0.005" ixy="0.0" ixz="0.0" iyy="0.005" iyz="0.0" izz="0.009"/>
-      </inertial-->
-      <!--libgazebo_ros_skid_steer_drive.so -->
-      <inertial>
-        <origin xyz="0 0 0" rpy="0 0 0"/>
-        <mass value="0.1"/>
-        <inertia ixx="0.0001" ixy="0.0" ixz="0.0" iyy="0.0001" iyz="0.0" izz="0.0001"/>
       </inertial>
       <visual>
@@ -52,8 +44,8 @@
     <gazebo reference="${prefix}_link">
       <material>Gazebo/White</material>
-      <mu1 value="2.5" />
-      <mu2 value="2.5" />
-      <kp value="50000" />
-      <kd value="10" />
+      <kp>1000000.0</kp>
+      <kd>100.0</kd>
+      <mu1>1.0</mu1>
+      <mu2>1.0</mu2>
       <minDepth>0.00</minDepth>
     </gazebo>
@@ -66,15 +58,8 @@
     </joint>
     <link name="body_link">
-      <!-- libgazebo_ros_planar_move.so -->
-      <!--inertial>
+      <inertial>
       <mass value="15.0"/>
       <origin xyz=" 0 0 0.1175"/>
-      <inertia ixx="0.13" ixy="0.0" ixz="0.0" iyy="0.33" iyz="0.0" izz="0.39"/>
-      </inertial-->
-      <!--libgazebo_ros_skid_steer_drive.so -->
-      <inertial>
-        <mass value="1.0"/>
-        <origin xyz=" 0 0 0.1175"/>
-        <inertia ixx="0.001" ixy="0.0" ixz="0.0" iyy="0.001" iyz="0.0" izz="0.001"/>
+      <inertia ixx="1" ixy="0.0" ixz="0.0" iyy="1" iyz="0.0" izz="1"/>
       </inertial>
       <visual>

File: racecar_simulator/urdf/racecar.xacro (robot description, xacro)
@@ -1,4 +1,9 @@
 <?xml version="1.0"?>
 <robot name="rrbot" xmlns:xacro="http://www.ros.org/wiki/xacro">
+  <xacro:arg name="robot_name" default="racecar"/>
+  <xacro:arg name="enable_odom_tf" default="true"/>
+  <xacro:arg name="odom_frame" default="odom"/>
+  <xacro:arg name="odom_topic" default="odom"/>
+  <xacro:arg name="cmd_topic" default="cmd_vel"/>
   <material name="white">
     <color rgba="1.0 1.0 1.0 1.0"/>
@@ -289,25 +294,29 @@
     <!--plugin filename="libgazebo_ros_skid_steer_drive.so" name="skid_steer_drive_controller">
       <updateRate>100.0</updateRate>
-      <robotNamespace></robotNamespace>
+      <robotNamespace>$(arg robot_name)</robotNamespace>
       <leftFrontJoint>front_left_wheel_joint</leftFrontJoint>
       <rightFrontJoint>front_right_wheel_joint</rightFrontJoint>
       <leftRearJoint>rear_left_wheel_joint</leftRearJoint>
       <rightRearJoint>rear_right_wheel_joint</rightRearJoint>
-      <wheelSeparation>0.34</wheelSeparation>
+      <covariance_x>0.000100</covariance_x>
+      <covariance_y>0.000100</covariance_y>
+      <covariance_yaw>0.010000</covariance_yaw>
+      <wheelSeparation>0.28</wheelSeparation>
       <wheelDiameter>0.135</wheelDiameter>
-      <robotBaseFrame>base_link</robotBaseFrame>
+      <robotBaseFrame>$(arg robot_name)/base_link</robotBaseFrame>
       <MaxForce>10.0</MaxForce>
       <torque>400</torque>
-      <commandTopic>cmd_vel</commandTopic>
-      <odometryTopic>odom</odometryTopic>
-      <odometryFrame>odom</odometryFrame>
-      <broadcastTF>1</broadcastTF>
+      <commandTopic>$(arg cmd_topic)</commandTopic>
+      <odometryTopic>$(arg odom_topic)</odometryTopic>
+      <odometryFrame>$(arg robot_name)/$(arg odom_frame)</odometryFrame>
+      <broadcastTF>$(arg enable_odom_tf)</broadcastTF>
     </plugin-->
-    <plugin name="object_controller" filename="libgazebo_ros_planar_move.so">
-      <commandTopic>cmd_vel</commandTopic>
-      <odometryTopic>odom</odometryTopic>
-      <odometryFrame>odom</odometryFrame>
+    <plugin name="object_controller" filename="libgazebo_ros_planar_move_drive.so">
+      <commandTopic>$(arg cmd_topic)</commandTopic>
+      <odometryTopic>$(arg odom_topic)</odometryTopic>
+      <odometryFrame>$(arg robot_name)/$(arg odom_frame)</odometryFrame>
       <odometryRate>100.0</odometryRate>
-      <robotBaseFrame>base_link</robotBaseFrame>
+      <robotBaseFrame>$(arg robot_name)/base_link</robotBaseFrame>
+      <broadcastTF>$(arg enable_odom_tf)</broadcastTF>
     </plugin>
   </gazebo>

File: racecar_simulator/urdf/racecar_robot.xacro (robot description, xacro)
@@ -5,4 +5,5 @@
   <xacro:arg name="odom_frame" default="odom"/>
   <xacro:arg name="odom_topic" default="odom"/>
+  <xacro:arg name="cmd_topic" default="cmd_vel"/>
   <xacro:include filename="$(find racecar_simulator)/urdf/move_macro.xacro"/>
   <xacro:include filename="$(find racecar_simulator)/urdf/laser_macro.xacro"/>
@@ -17,5 +18,5 @@
   <xacro:imu_macro prefix="imu" parent="base_link" xyz="0.16575 0 0.168" robot_name="$(arg robot_name)"/>
   <gazebo>
-    <plugin filename="libgazebo_ros_skid_steer_drive.so" name="skid_steer_drive_controller">
+    <!--plugin filename="libgazebo_ros_skid_steer_drive.so" name="skid_steer_drive_controller">
       <updateRate>100.0</updateRate>
       <robotNamespace>$(arg robot_name)</robotNamespace>
@@ -32,15 +33,21 @@
       <MaxForce>10.0</MaxForce>
       <torque>400</torque>
-      <commandTopic>cmd_vel</commandTopic>
+      <commandTopic>$(arg cmd_topic)</commandTopic>
       <odometryTopic>$(arg odom_topic)</odometryTopic>
       <odometryFrame>$(arg robot_name)/$(arg odom_frame)</odometryFrame>
       <broadcastTF>$(arg enable_odom_tf)</broadcastTF>
-    </plugin>
-    <!--plugin name="object_controller" filename="libgazebo_ros_planar_move.so">
-      <commandTopic>cmd_vel</commandTopic>
-      <odometryTopic>odom</odometryTopic>
-      <odometryFrame>$(arg robot_name)/odom</odometryFrame>
+    </plugin-->
+    <plugin name="object_controller" filename="libgazebo_ros_planar_move_drive.so">
+      <commandTopic>$(arg cmd_topic)</commandTopic>
+      <odometryTopic>$(arg odom_topic)</odometryTopic>
+      <odometryFrame>$(arg robot_name)/$(arg odom_frame)</odometryFrame>
       <odometryRate>100.0</odometryRate>
       <robotBaseFrame>$(arg robot_name)/base_link</robotBaseFrame>
+      <broadcastTF>$(arg enable_odom_tf)</broadcastTF>
+    </plugin>
+    <!--plugin name="gazebo_ros_control" filename="libgazebo_ros_control.so">
+      <robotNamespace>$(arg robot_name)</robotNamespace>
+      <robotSimType>gazebo_ros_control/DefaultRobotHWSim</robotSimType>
+      <legacyModeNS>true</legacyModeNS>
     </plugin-->
   </gazebo>
