Commit message: fix the bug in move_base and navigation is totally completed

File: racecar_simulator/urdf/imu_macro.xacro (robot description, xacro)
@@ -1,5 +1,5 @@
 <?xml version="1.0"?>
 <robot name="racecar" xmlns:xacro="http://ros.org/wiki/xacro">
-  <xacro:macro name="imu_macro" params="parent prefix xyz robot_name">
+  <xacro:macro name="imu_macro" params="parent prefix xyz robot_namespace">
     <joint name="imu_joint" type="fixed">
       <parent link="${parent}"/>
@@ -33,9 +33,9 @@
           <topicName>${prefix}/data</topicName>
           <bodyName>${prefix}_link</bodyName>
-          <updateRateHZ>10.0</updateRateHZ>
+          <updateRateHZ>100.0</updateRateHZ>
           <gaussianNoise>0.0</gaussianNoise>
           <xyzOffset>0 0 0</xyzOffset>
           <rpyOffset>0 0 0</rpyOffset>
-          <frameName>${robot_name}/${prefix}_link</frameName>
+          <frameName>${robot_namespace}/${prefix}_link</frameName>
         </plugin>
         <pose>0 0 0 0 0 0</pose>

File: racecar_simulator/urdf/racecar.xacro (robot description, xacro)
@@ -315,7 +315,7 @@
       <commandTopic>$(arg cmd_topic)</commandTopic>
       <odometryTopic>$(arg odom_topic)</odometryTopic>
-      <odometryFrame>$(arg robot_name)/$(arg odom_frame)</odometryFrame>
+      <odometryFrame>$(arg odom_frame)</odometryFrame>
       <odometryRate>100.0</odometryRate>
-      <robotBaseFrame>$(arg robot_name)/base_link</robotBaseFrame>
+      <robotBaseFrame>base_link</robotBaseFrame>
       <broadcastTF>$(arg enable_odom_tf)</broadcastTF>
     </plugin>

File: racecar_simulator/urdf/racecar_robot.xacro (robot description, xacro)
@@ -1,5 +1,5 @@
 <?xml version="1.0"?>
 <robot name="racecar" xmlns:xacro="http://ros.org/wiki/xacro">
-  <xacro:arg name="robot_name" default="racecar"/>
+  <xacro:arg name="robot_namespace" default="racecar"/>
   <xacro:arg name="enable_odom_tf" default="true"/>
   <xacro:arg name="odom_frame" default="odom"/>
@@ -16,9 +16,9 @@
   <xacro:wheel_macro prefix="rear_left_wheel" parent="base_link" xyz="-0.1575 0.14 0.0675"/>
   <xacro:laser_macro prefix="laser" parent="base_link" xyz="0.07 0 0.2575"/>
-  <xacro:imu_macro prefix="imu" parent="base_link" xyz="0.16575 0 0.168" robot_name="$(arg robot_name)"/>
+  <xacro:imu_macro prefix="imu" parent="base_link" xyz="0.16575 0 0.168" robot_namespace="$(arg robot_namespace)"/>
   <gazebo>
     <!--plugin filename="libgazebo_ros_skid_steer_drive.so" name="skid_steer_drive_controller">
       <updateRate>100.0</updateRate>
-      <robotNamespace>$(arg robot_name)</robotNamespace>
+      <robotNamespace>$(arg robot_namespace)</robotNamespace>
       <leftFrontJoint>front_left_wheel_joint</leftFrontJoint>
       <rightFrontJoint>front_right_wheel_joint</rightFrontJoint>
@@ -30,10 +30,10 @@
       <wheelSeparation>0.28</wheelSeparation>
       <wheelDiameter>0.135</wheelDiameter>
-      <robotBaseFrame>$(arg robot_name)/base_link</robotBaseFrame>
+      <robotBaseFrame>$(arg robot_namespace)/base_link</robotBaseFrame>
       <MaxForce>10.0</MaxForce>
       <torque>400</torque>
       <commandTopic>$(arg cmd_topic)</commandTopic>
       <odometryTopic>$(arg odom_topic)</odometryTopic>
-      <odometryFrame>$(arg robot_name)/$(arg odom_frame)</odometryFrame>
+      <odometryFrame>$(arg robot_namespace)/$(arg odom_frame)</odometryFrame>
       <broadcastTF>$(arg enable_odom_tf)</broadcastTF>
     </plugin-->
@@ -41,11 +41,11 @@
       <commandTopic>$(arg cmd_topic)</commandTopic>
       <odometryTopic>$(arg odom_topic)</odometryTopic>
-      <odometryFrame>$(arg robot_name)/$(arg odom_frame)</odometryFrame>
+      <odometryFrame>$(arg robot_namespace)/$(arg odom_frame)</odometryFrame>
       <odometryRate>100.0</odometryRate>
-      <robotBaseFrame>$(arg robot_name)/base_link</robotBaseFrame>
+      <robotBaseFrame>$(arg robot_namespace)/base_link</robotBaseFrame>
       <broadcastTF>$(arg enable_odom_tf)</broadcastTF>
     </plugin>
     <!--plugin name="gazebo_ros_control" filename="libgazebo_ros_control.so">
-      <robotNamespace>$(arg robot_name)</robotNamespace>
+      <robotNamespace>$(arg robot_namespace)</robotNamespace>
       <robotSimType>gazebo_ros_control/DefaultRobotHWSim</robotSimType>
       <legacyModeNS>true</legacyModeNS>

Commit message: simplify the launch files

File: racecar_simulator/urdf/imu_macro.xacro (robot description, xacro)
@@ -1,5 +1,5 @@
 <?xml version="1.0"?>
-<robot name="racecar" xmlns:xacro="http://ros.org/wiki/xacro">
-  <xacro:macro name="imu_macro" params="parent prefix xyz robot_namespace">
+<robot name="racecar" xmlns:xacro="http://www.ros.org/wiki/xacro">
+  <xacro:macro name="imu_macro" params="parent prefix xyz">
     <joint name="imu_joint" type="fixed">
       <parent link="${parent}"/>
@@ -29,7 +29,7 @@
         <update_rate>100</update_rate>
         <visualize>true</visualize>
-        <topic>data</topic>
+        <topic>__default_topic__</topic>
         <plugin name="gazebo_ros_imu_controller" filename="libgazebo_ros_imu_sensor.so">
-          <topicName>${prefix}/data</topicName>
+          <topicName>/${prefix}/data</topicName>
           <bodyName>${prefix}_link</bodyName>
           <updateRateHZ>10.0</updateRateHZ>
@@ -37,5 +37,5 @@
           <xyzOffset>0 0 0</xyzOffset>
           <rpyOffset>0 0 0</rpyOffset>
-          <frameName>${robot_namespace}/${prefix}_link</frameName>
+          <frameName>${prefix}_link</frameName>
         </plugin>
         <pose>0 0 0 0 0 0</pose>

File: racecar_simulator/urdf/laser_macro.xacro (robot description, xacro)
@@ -1,4 +1,4 @@
 <?xml version="1.0"?>
-<robot name="racecar" xmlns:xacro="http://ros.org/wiki/xacro">
+<robot name="racecar" xmlns:xacro="http://www.ros.org/wiki/xacro">
   <xacro:macro name="laser_macro" params="parent prefix xyz">
     <joint name="${prefix}_joint" type="fixed">
@@ -49,5 +49,5 @@
         </ray>
         <plugin name="gazebo_ros_laser_controller" filename="libgazebo_ros_laser.so">
-          <topicName>${prefix}/scan</topicName>
+          <topicName>/${prefix}/scan</topicName>
           <frameName>${prefix}_link</frameName>
         </plugin>

File: racecar_simulator/urdf/racecar_robot.xacro (robot description, xacro)
@@ -1,5 +1,4 @@
 <?xml version="1.0"?>
-<robot name="racecar" xmlns:xacro="http://ros.org/wiki/xacro">
-  <xacro:arg name="robot_namespace" default="racecar"/>
+<robot name="racecar" xmlns:xacro="http://www.ros.org/wiki/xacro">
   <xacro:arg name="enable_odom_tf" default="true"/>
   <xacro:arg name="odom_frame" default="odom"/>
@@ -16,9 +15,9 @@
   <xacro:wheel_macro prefix="rear_left_wheel" parent="base_link" xyz="-0.1575 0.14 0.0675"/>
   <xacro:laser_macro prefix="laser" parent="base_link" xyz="0.07 0 0.2575"/>
-  <xacro:imu_macro prefix="imu" parent="base_link" xyz="0.16575 0 0.168" robot_namespace="$(arg robot_namespace)"/>
+  <xacro:imu_macro prefix="imu" parent="base_link" xyz="0.16575 0 0.168"/>
   <gazebo>
     <!--plugin filename="libgazebo_ros_skid_steer_drive.so" name="skid_steer_drive_controller">
       <updateRate>100.0</updateRate>
-      <robotNamespace>$(arg robot_namespace)</robotNamespace>
+      <robotNamespace>""</robotNamespace>
       <leftFrontJoint>front_left_wheel_joint</leftFrontJoint>
       <rightFrontJoint>front_right_wheel_joint</rightFrontJoint>
@@ -30,10 +29,10 @@
       <wheelSeparation>0.28</wheelSeparation>
       <wheelDiameter>0.135</wheelDiameter>
-      <robotBaseFrame>$(arg robot_namespace)/base_link</robotBaseFrame>
+      <robotBaseFrame>base_link</robotBaseFrame>
       <MaxForce>10.0</MaxForce>
       <torque>400</torque>
       <commandTopic>$(arg cmd_topic)</commandTopic>
       <odometryTopic>$(arg odom_topic)</odometryTopic>
-      <odometryFrame>$(arg robot_namespace)/$(arg odom_frame)</odometryFrame>
+      <odometryFrame>$(arg odom_frame)</odometryFrame>
       <broadcastTF>$(arg enable_odom_tf)</broadcastTF>
     </plugin-->
@@ -41,14 +40,9 @@
       <commandTopic>$(arg cmd_topic)</commandTopic>
       <odometryTopic>$(arg odom_topic)</odometryTopic>
-      <odometryFrame>$(arg robot_namespace)/$(arg odom_frame)</odometryFrame>
+      <odometryFrame>$(arg odom_frame)</odometryFrame>
       <odometryRate>100.0</odometryRate>
-      <robotBaseFrame>$(arg robot_namespace)/base_link</robotBaseFrame>
+      <robotBaseFrame>base_link</robotBaseFrame>
       <broadcastTF>$(arg enable_odom_tf)</broadcastTF>
     </plugin>
-    <!--plugin name="gazebo_ros_control" filename="libgazebo_ros_control.so">
-      <robotNamespace>$(arg robot_namespace)</robotNamespace>
-      <robotSimType>gazebo_ros_control/DefaultRobotHWSim</robotSimType>
-      <legacyModeNS>true</legacyModeNS>
-    </plugin-->
   </gazebo>
 </robot>
